File: Caps32Project.kicad_pcb (KiCad board)
At the start: 2 copper layers, 20 x 33 mm, 23 parts, among them J1 Ph 2.0, J2 Sh 1.0, P1 USB_C_Plug_USB2.0, Q1 AO3401A, U1 MPU-6050, U2 MAX17048G_T10, U3 ESP32C3_SuperMini, U4 MCP73831-2-OT

Commit message: LGTM
Parts:
- added C6: 1.0uF, Capacitor_SMD:C_0402_1005Metric_Pad0.74x0.62mm_HandSolder, F.Cu at (187.0, 56.8)
- added D3: WS2812B, LED_SMD:LED_WS2812B_PLCC4_5.0x5.0mm_P3.2mm, F.Cu at (194.8, 68.2)
- moved C13 11.9 mm to (190.0, 67.8)
- moved R2 10.6 mm to (188.8, 60.2)
- moved R5 8.53 mm to (189.5, 55.2), turned to -90 degrees
- moved D6 7.89 mm to (188.2, 50.5)
- moved D1 7.23 mm to (187.8, 55.0), turned to 0 degrees
- moved R3 7.00 mm to (190.0, 59.0), turned to 180 degrees
- moved C4 6.25 mm to (195.5, 59.5), turned to 180 degrees
- moved C1 5.21 mm to (187.0, 59.4), turned to 90 degrees
- moved R1 4.33 mm to (188.2, 56.8), turned to 90 degrees
- moved U2 4.27 mm to (196.2, 62.7)
- moved Q1 4.18 mm to (188.2, 62.8), turned to 90 degrees
- moved J2 4.00 mm to (194.0, 50.0)
- moved D2 3.61 mm to (189.5, 66.0), turned to 90 degrees
- moved C3 3.10 mm to (190.0, 57.8)
- moved U4 2.91 mm to (191.9, 62.6)
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Connections:
- U3 pad 10: unconnected-(U3-GPIO10-Pad10) -> RGB
Routing:
- net SCL: track 31.1 -> 17.2 mm, vias 3 -> 2
- net +3V3: track 21.7 -> 34.3 mm, vias 0 -> 2
- net SDA: track 26.9 -> 16.6 mm
- net +BATT: track 21.9 -> 31.5 mm, vias 2 -> 0
- net VBUS: track 31.4 -> 40.2 mm
- net RGB: track 0.00 -> 6.92 mm
- net GND: track 29.0 -> 34.3 mm, vias 14 -> 11
- net Net-(D2-A): track 1.51 -> 5.45 mm
- net +5V: track 29.2 -> 25.3 mm
- net Net-(D2-K): track 2.62 -> 3.42 mm
- net Net-(U4-PROG): track 1.98 -> 2.67 mm

Commit message: Tweak
Parts:
- removed U4: MCP73831-2-OT, Package_TO_SOT_SMD:SOT-23-5
- added C10: 10uF, Capacitor_SMD:C_0402_1005Metric_Pad0.74x0.62mm_HandSolder, F.Cu at (237.8, 56.1)
- added C11: 10uF, Capacitor_SMD:C_0402_1005Metric_Pad0.74x0.62mm_HandSolder, F.Cu at (241.0, 48.2)
- added C12: 10uF, Capacitor_SMD:C_0402_1005Metric_Pad0.74x0.62mm_HandSolder, F.Cu at (241.0, 50.2)
- added C14: 10uF, Capacitor_SMD:C_0402_1005Metric_Pad0.74x0.62mm_HandSolder, F.Cu at (241.0, 54.1)
- added C7: 10uF, Capacitor_SMD:C_0402_1005Metric_Pad0.74x0.62mm_HandSolder, F.Cu at (237.8, 50.2)
- added C8: 10uF, Capacitor_SMD:C_0402_1005Metric_Pad0.74x0.62mm_HandSolder, F.Cu at (237.8, 52.1)
- added C9: 10uF, Capacitor_SMD:C_0402_1005Metric_Pad0.74x0.62mm_HandSolder, F.Cu at (237.8, 54.1)
- added D4: LED, LED_SMD:LED_0402_1005Metric_Pad0.77x0.64mm_HandSolder, B.Cu at (188.0, 78.2)
- added D5: LED, LED_SMD:LED_0402_1005Metric_Pad0.77x0.64mm_HandSolder, B.Cu at (187.0, 78.2)
- added D7: LED, LED_SMD:LED_0402_1005Metric_Pad0.77x0.64mm_HandSolder, B.Cu at (186.0, 78.2)
- added L1: 1R0, Inductor_SMD:L_6.3x6.3_H3, F.Cu at (196.2, 75.0)
- added R4: 10K, Resistor_SMD:R_0402_1005Metric_Pad0.72x0.64mm_HandSolder, F.Cu at (234.6, 64.0)
- C1, C2: value 4.7uF -> 10uF
- C5: value 1.0uF -> 10uF
- D2: moved to B.Cu
- P1: footprint Connector_USB:USB_C_Receptacle_XKB_U262-16XN-4BVC11 -> Connector_USB:USB_C_Receptacle_Palconn_UTC16-G
- R2: value 1K -> 2R
- R3: value 2K -> 2R
- U2: value MAX17048G_T10 -> IP5306; footprint Custom:SON50P200X200X80-9N -> Custom:IP5306
- moved C13 53.3 mm to (241.0, 52.1)
- moved C6 51.5 mm to (237.8, 48.2), turned to 0 degrees
- moved R7 49.5 mm to (234.6, 70.0), turned to 0 degrees
- moved C1 48.9 mm to (234.6, 48.2), turned to 0 degrees
- moved R6 47.1 mm to (234.6, 68.0), turned to 0 degrees
- moved R1 46.4 mm to (234.6, 58.1), turned to 0 degrees
- moved R5 46.4 mm to (234.6, 66.0), turned to 0 degrees
- moved R2 45.8 mm to (234.6, 60.0)
- moved C2 45.3 mm to (234.6, 50.2)
- moved C3 44.9 mm to (234.6, 52.1)
- moved R3 44.7 mm to (234.6, 62.0), turned to 0 degrees
- moved C5 42.1 mm to (234.6, 56.1), turned to 0 degrees
- moved C4 39.4 mm to (234.6, 54.1), turned to 0 degrees
- moved D2 12.2 mm to (189.0, 78.2), turned to -90 degrees
- moved D1 10.5 mm to (188.8, 65.5)
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Connections:
- C1 pad 1: VBUS -> GND
- C1 pad 2: GND -> Net-(C1-Pad2)
- C2 pad 1: +BATT -> VBUS
- C5 pad 1: +BATT -> GND
- C5 pad 2: GND -> Net-(C5-Pad2)
- R2 pad 2: Net-(D2-A) -> Net-(C1-Pad2)
- R3 pad 1: Net-(U4-PROG) -> +BATT
- R3 pad 2: GND -> Net-(C5-Pad2)
- U2 pad 1: GND -> VBUS
- U2 pad 2: +BATT -> Net-(D2-A)
- U2 pad 3: +BATT -> Net-(D5-A)
- U2 pad 4: GND -> Net-(D2-K)
- U2 pad 5: unconnected-(U2-~{ALERT}-Pad5) -> Net-(U2-KEY)
- U2 pad 6: GND -> +BATT
- U2 pad 7: SCL -> Net-(U2-SW)
- U2 pad 8: SDA -> VCC
Routing:
- net VBUS: track 40.2 -> 0.00 mm, vias 2 -> 0
- net GND: track 34.3 -> 0.00 mm, vias 11 -> 0
- net +3V3: track 34.3 -> 0.00 mm, vias 2 -> 0
- net +BATT: track 31.5 -> 0.00 mm
- net +5V: track 25.3 -> 0.00 mm, vias 2 -> 0
- net SCL: track 17.2 -> 0.00 mm, vias 2 -> 0
- net SDA: track 16.6 -> 0.00 mm, vias 2 -> 0
- net RGB: track 6.92 -> 0.00 mm
- net Net-(D2-A): track 5.45 -> 0.00 mm
- net Net-(D2-K): track 3.42 -> 0.00 mm
- net Net-(U1-CPOUT): track 3.32 -> 0.00 mm
- net Net-(P1-CC2): track 2.87 -> 0.00 mm
- net Net-(U4-PROG): track 2.67 -> 0.00 mm
- net Net-(P1-CC1): track 2.44 -> 0.00 mm
- net Net-(U1-REGOUT): track 2.13 -> 0.00 mm
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- removed copper zone on B.Cu, net GND

Commit message: Non Latch
Parts:
- D6: moved to B.Cu
- moved C1 52.8 mm to (186.8, 70.5), turned to 180 degrees
- moved C13 52.4 mm to (191.5, 69.2)
- moved C2 51.8 mm to (186.2, 68.8), turned to 90 degrees
- moved R5 50.5 mm to (184.2, 69.5), turned to 180 degrees
- moved R7 50.4 mm to (184.2, 70.8), turned to 180 degrees
- moved R2 47.6 mm to (187.8, 68.8), turned to -90 degrees
- moved R1 47.4 mm to (187.2, 56.0)
- moved C6 47.4 mm to (190.4, 48.2)
- moved C14 47.2 mm to (194.0, 58.8), turned to 180 degrees
- moved C4 47.2 mm to (187.4, 54.8), turned to 180 degrees
- moved C3 46.6 mm to (188.2, 48.2)
- moved C11 46.4 mm to (196.5, 61.5)
- moved C12 46.3 mm to (195.8, 59.8), turned to 90 degrees
- moved R6 45.9 mm to (188.8, 70.0), turned to 90 degrees
- moved C7 45.0 mm to (197.2, 69.8), turned to 90 degrees
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Connections:
- Q1 pad 3: +BATT -> VCC
Routing:
- net VBUS: track 0.00 -> 30.6 mm, vias 0 -> 1
- net +3V3: track 0.00 -> 27.6 mm
- net +5V: track 0.00 -> 27.2 mm, vias 0 -> 2
- net SCL: track 0.00 -> 21.2 mm, vias 0 -> 2
- net +BATT: track 0.00 -> 19.4 mm
- net SDA: track 0.00 -> 18.3 mm, vias 0 -> 2
- net VCC: track 0.00 -> 17.1 mm
- net Net-(D2-A): track 0.00 -> 16.1 mm, vias 0 -> 1
- net Net-(D2-K): track 0.00 -> 14.5 mm, vias 0 -> 1
- net Net-(D5-A): track 0.00 -> 14.0 mm, vias 0 -> 1
- net RGB: track 0.00 -> 11.4 mm
- net GND: track 0.00 -> 10.7 mm, vias 0 -> 22
- net Net-(U2-SW): track 0.00 -> 8.66 mm
- net Net-(P1-CC1): track 0.00 -> 2.66 mm
- net Net-(P1-CC2): track 0.00 -> 2.22 mm
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- added copper zone on B.Cu, net GND

Commit message: Tweak
Parts:
- D2, D4, D5, D6, D7, J1: moved to F.Cu
- D3, R6, R7: moved to B.Cu
- U3: footprint Custom:ESP32C3_Supermini_THT -> Custom:Supermini_Custom
- moved R4 171.0 mm to (30.2, 27.7)
- moved D6 167.4 mm to (29.6, 46.0), turned to 180 degrees
- moved J2 166.7 mm to (29.1, 38.8), turned to -90 degrees
- moved C11 165.8 mm to (31.2, 48.5), turned to 180 degrees
- moved C5 165.3 mm to (36.1, 48.5)
- moved L1 164.5 mm to (36.1, 37.8)
- moved C12 164.3 mm to (32.2, 43.5), turned to 180 degrees
- moved R3 163.8 mm to (38.4, 48.2), turned to 180 degrees
- moved J1 163.7 mm to (38.3, 54.5), turned to 90 degrees
- moved R2 162.4 mm to (27.3, 43.5), turned to 0 degrees
- moved C6 161.3 mm to (29.8, 33.2), turned to 90 degrees
- moved C10 160.8 mm to (34.0, 43.0), turned to 90 degrees
- moved C7 160.2 mm to (38.3, 49.5), turned to 0 degrees
- moved C9 160.0 mm to (35.0, 43.0), turned to 90 degrees
- moved U2 160.0 mm to (37.8, 28.8), turned to 90 degrees
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Routing:
- net GND: track 10.7 -> 63.5 mm, vias 22 -> 11
- net +3V3: track 27.6 -> 51.1 mm, vias 0 -> 2
- net VCC: track 17.1 -> 39.6 mm, vias 0 -> 2
- net +BATT: track 19.4 -> 32.7 mm
- net SDA: track 18.3 -> 30.3 mm, vias 2 -> 4
- net Net-(D5-A): track 14.0 -> 2.72 mm, vias 1 -> 0
- net VBUS: track 30.6 -> 41.2 mm, vias 1 -> 4
- net Net-(D2-K): track 14.5 -> 6.47 mm, vias 1 -> 0
- net Net-(D2-A): track 16.1 -> 10.5 mm, vias 1 -> 0
- net SCL: track 21.2 -> 26.5 mm, vias 2 -> 4
- net Net-(U2-KEY): track 1.87 -> 4.75 mm
- net RGB: track 11.4 -> 13.1 mm, vias 0 -> 2
- net +5V: track 27.2 -> 25.9 mm, vias 2 -> 1
- net Net-(C1-Pad2): track 2.04 -> 1.27 mm
- net Net-(U1-REGOUT): track 1.30 -> 2.06 mm
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Other:
- board size 20 x 33 mm -> 20 x 32 mm

Commit message: Fixing
Parts:
- added SW1: SW_Push, Button_Switch_SMD:SW_Push_1TS009xxxx-xxxx-xxxx_6x6x5mm, B.Cu at (33.6, 55.8)
- J1: footprint Connector_JST:JST_PH_S2B-PH-K_1x02_P2.00mm_Horizontal -> Connector_JST:JST_PH_S2B-PH-SM4-TB_1x02-1MP_P2.00mm_Horizontal
- R6, R7: moved to F.Cu
- moved C6 24.9 mm to (35.6, 57.4)
- moved R4 19.4 mm to (33.4, 46.8)
- moved R1 18.8 mm to (32.0, 57.4)
- moved D1 17.5 mm to (33.8, 56.8), turned to 180 degrees
- moved C3 17.2 mm to (34.0, 58.8), turned to 180 degrees
- moved U1 17.2 mm to (28.8, 56.6), turned to 0 degrees
- moved J1 15.4 mm to (31.1, 41.0), turned to -90 degrees
- moved R2 14.3 mm to (40.4, 49.2)
- moved C1 14.2 mm to (42.8, 49.2)
- moved R6 12.8 mm to (44.8, 50.2)
- moved D6 12.6 mm to (42.2, 46.6)
- moved R7 12.6 mm to (42.4, 50.4)
- moved R5 12.3 mm to (39.2, 50.4)
- moved P1 11.4 mm to (42.3, 54.9)
- moved J2 10.9 mm to (29.4, 49.6)
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Connections:
- R4 pad 1: GND -> Net-(R4-Pad1)
Routing:
- net GND: track 63.5 -> 28.5 mm, vias 11 -> 14
- net Net-(U2-KEY): track 4.75 -> 26.2 mm
- net +5V: track 25.9 -> 36.7 mm
- net VBUS: track 41.2 -> 31.2 mm, vias 4 -> 0
- net RGB: track 13.1 -> 22.2 mm, vias 2 -> 0
- net VCC: track 39.6 -> 30.9 mm, vias 2 -> 0
- net +BATT: track 32.7 -> 24.3 mm, vias 0 -> 2
- net Net-(R4-Pad1): track 0.00 -> 5.49 mm, vias 0 -> 1
- net +3V3: track 51.1 -> 56.4 mm, vias 2 -> 1
- net Net-(U1-REGOUT): track 2.06 -> 5.25 mm
- net Net-(U2-SW): track 8.91 -> 6.80 mm, vias 0 -> 2
- net Net-(D5-A): track 2.72 -> 4.73 mm
- net Net-(U1-CPOUT): track 1.38 -> 3.31 mm
- net SDA: track 30.3 -> 28.4 mm, vias 4 -> 1
- net Net-(P1-CC2): track 1.91 -> 2.78 mm, vias 1 -> 0
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Other:
- board size 20 x 32 mm -> 22.5 x 35 mm

Commit message: T
Parts:
- C12: moved to B.Cu
- moved D7 9.36 mm to (37.4, 27.0), turned to -90 degrees
- moved D5 7.87 mm to (38.5, 27.0), turned to 90 degrees
- moved U2 6.71 mm to (33.8, 32.2), turned to 180 degrees
- moved D2 6.32 mm to (39.8, 27.0), turned to -90 degrees
- moved D4 5.03 mm to (41.0, 27.0), turned to 90 degrees
- moved C12 0.45 mm to (35.0, 35.4)
Routing:
- net Net-(U2-KEY): track 26.2 -> 11.8 mm
- net VCC: track 30.9 -> 17.2 mm, vias 0 -> 1
- net VBUS: track 31.2 -> 42.5 mm
- net +BATT: track 24.3 -> 15.3 mm, vias 2 -> 0
- net Net-(D2-K): track 7.22 -> 11.0 mm
- net Net-(D2-A): track 11.2 -> 7.94 mm, vias 0 -> 2
- net Net-(U2-SW): track 6.80 -> 9.40 mm, vias 2 -> 0
- net Net-(D5-A): track 4.73 -> 7.30 mm, vias 0 -> 2
- net +5V: track 36.7 -> 37.1 mm, vias 1 -> 3
- net GND: vias 14 -> 13

Commit message: t
Routing:
- net +5V: track 37.1 -> 35.1 mm
- net VBUS: track 42.5 -> 43.2 mm
- net RGB: track 22.2 -> 22.9 mm
Changed lines of the file:
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@@
 		)
 		(property "Value" "IP5306"
-			(at 3.175 -1.143 360)
+			(at 3.175 -1.143 0)
 			(layer "F.Fab")
 			(hide yes)
@@
 		)
 		(property "Footprint" "Custom:IP5306"
-			(at 0 0 360)
+			(at 0 0 0)
 			(layer "F.Fab")
 			(hide yes)
@@
 		)
 		(property "Datasheet" ""
-			(at 0 0 360)
+			(at 0 0 0)
 			(layer "F.Fab")
 			(hide yes)
@@
 		)
 		(property "Description" ""
-			(at 0 0 360)
+			(at 0 0 0)
 			(layer "F.Fab")
 			(hide yes)
@@
 		(tags "capacitor handsolder")
 		(property "Reference" "C12"
-			(at 0 1.16 360)
+			(at 0 1.16 0)
 			(layer "B.SilkS")
 			(hide yes)
@@
 		)
 		(property "Value" "10uF"
-			(at 0 -1.16 360)
+			(at 0 -1.16 0)
 			(layer "B.Fab")
 			(hide yes)
@@
 		)
 		(fp_text user "${REFERENCE}"
-			(at 0 0 360)
+			(at 0 0 0)
 			(layer "B.Fab")
 			(effects
@@
 	)
 	(segment
-		(start 44.2 46.6)
-		(end 44.2 44.3675)
+		(start 41.8 42.4)
+		(end 41.8 41.5)
 		(width 0.2)
 		(layer "F.Cu")
@@
 	)
 	(segment
-		(start 42.5 41.5)
-		(end 41.8 41.5)
+		(start 44.2 46.6)
+		(end 44.2 44.3675)
 		(width 0.2)
 		(layer "F.Cu")
@@
 	)
 	(segment
-		(start 42.4 32.2)
-		(end 42.4 40.2)
+		(start 41.824265 42.424265)
+		(end 41.8 42.4)
 		(width 0.2)
 		(layer "F.Cu")
@@
 	)
 	(segment
-		(start 42.8375 41.8375)
-		(end 42.5 41.5)
+		(start 42.4 32.2)
+		(end 42.4 40.2)
 		(width 0.2)
 		(layer "F.Cu")
@@
 	)
 	(segment
-		(start 42.8375 44.3625)
-		(end 42.8375 41.8375)
-		(width 0.2)
-		(layer "F.Cu")
-		(net 9)
-	)
-	(segment
-		(start 41.6 44.6)
-		(end 42.6 44.6)
-		(width 0.2)
-		(layer "F.Cu")
-		(net 9)
-	)
-	(segment
 		(start 42.2 32)
 		(end 42.4 32.2)
@@
 	)
 	(segment
-		(start 42.6 44.6)
-		(end 42.8375 44.3625)
-		(width 0.2)
-		(layer "F.Cu")
-		(net 9)
-	)
-	(segment
 		(start 41.8 40.8)
 		(end 41.8 41.5)
@@
 	)
 	(via
-		(at 41.6 44.6)
+		(at 41.824265 42.424265)
 		(size 0.6)
 		(drill 0.3)
@@
 	)
 	(segment
-		(start 42.4 47)
-		(end 41.6 46.2)
+		(start 41.824265 42.424265)
+		(end 41.824265 46.424265)
 		(width 0.2)
 		(layer "B.Cu")
@@
 	)
 	(segment
-		(start 41.6 46.2)
-		(end 41.6 44.6)
+		(start 41.824265 46.424265)
+		(end 42.4 47)
 		(width 0.2)
 		(layer "B.Cu")
@@
 	)
 	(segment
-		(start 40.448529 29.4)
-		(end 43.2375 32.188971)
+		(start 39.8 52.335)
+		(end 39.88 52.415)
 		(width 0.2)
 		(layer "F.Cu")
@@
 	)
 	(segment
-		(start 39.8 52.335)
-		(end 39.88 52.415)
+		(start 40.04 52.575)
+		(end 40.04 53.255)
 		(width 0.2)
 		(layer "F.Cu")
@@
 	)
 	(segment
-		(start 40.04 52.575)
-		(end 40.04 53.255)
+		(start 35.705 29.4)
+		(end 42 29.4)
+		(width 0.2)
+		(layer "F.Cu")
+		(net 27)
+	)
+	(segment
+		(start 43 45.05)
+		(end 41.45 46.6)
+		(width 0.2)
+		(layer "F.Cu")
+		(net 27)
+	)
+	(segment
+		(start 43 30.4)
+		(end 43 45.05)
 		(width 0.2)
 		(layer "F.Cu")
@@
 	)
 	(segment
+		(start 42 29.4)
+		(end 43 30.4)
+		(width 0.2)
+		(layer "F.Cu")
+		(net 27)
+	)
+	(segment
 		(start 44.48 52.615)
 		(end 44.68 52.415)
@@
 	)
 	(segment
-		(start 39.8025 49.2)
-		(end 39.8025 50.3975)
+		(start 41.45 46.6)
+		(end 40.2 46.6)
 		(width 0.2)
 		(layer "F.Cu")
@@
 	)
 	(segment
-		(start 41.8 43.4)
-		(end 40.2 45)
+		(start 39.8025 49.2)
+		(end 39.8025 50.3975)
 		(width 0.2)
 		(layer "F.Cu")
@@
 	)
 	(segment
-		(start 43.2375 44.8125)
-		(end 41.45 46.6)
+		(start 41.8 43.4)
+		(end 40.2 45)
 		(width 0.2)
 		(layer "F.Cu")
@@
 	)
 	(segment
-		(start 43.2375 32.188971)
-		(end 43.2375 44.8125)
-		(width 0.2)
-		(layer "F.Cu")
-		(net 27)
-	)
-	(segment
-		(start 41.45 46.6)
-		(end 40.2 46.6)
-		(width 0.2)
-		(layer "F.Cu")
-		(net 27)
-	)
-	(segment
 		(start 44.48 53.295)
 		(end 44.48 52.615)
@@
 	)
 	(segment
-		(start 35.705 29.4)
-		(end 40.448529 29.4)
-		(width 0.2)
-		(layer "F.Cu")
-		(net 27)
-	)
-	(segment
 		(start 39.88 52.415)
 		(end 40.04 52.575)
@@
 	)
 	(segment
-		(start 36 47.4)
-		(end 41.36 42.04)
+		(start 36.6 55.2)
+		(end 36 54.6)
 		(width 0.2)
 		(layer "B.Cu")
@@
 	)
 	(segment
-		(start 36.6 55.2)
-		(end 36 54.6)
+		(start 36 54.6)
+		(end 36 47.4)
 		(width 0.2)
 		(layer "B.Cu")
@@
 	)
 	(segment
-		(start 41.36 42.04)
-		(end 44.6275 42.04)
+		(start 36 47.4)
+		(end 42.2 41.2)
 		(width 0.2)
 		(layer "B.Cu")
@@
 	)
 	(segment
-		(start 36 54.6)
-		(end 36 47.4)
+		(start 42.2 41.2)
+		(end 43.7875 41.2)
+		(width 0.2)
+		(layer "B.Cu")
+		(net 35)
+	)
+	(segment
+		(start 43.7875 41.2)
+		(end 44.6275 42.04)
 		(width 0.2)
 		(layer "B.Cu")
