File: BMI.kicad_sch (KiCad schematic)
At the start: 25 parts, among them Q4 BSS138, Q5 BSS138, U10 BMI160/270, U7 MAX30102, U8 LN1134A182MR-G, U9 BMM150

Commit message: Update Board
Parts:
- removed C20: 100nF 16V, Capacitor_SMD:C_0603_1608Metric, symbol Device:C_Small
- removed JP1, JP2: SolderJumper_3_Bridged12, Jumper:SolderJumper-3_P1.3mm_Bridged2Bar12_RoundedPad1.0x1.5mm, symbol Jumper:SolderJumper_3_Bridged12
- removed TP12: INT, TestPoint:TestPoint_Pad_D1.0mm, symbol Connector:TestPoint
- removed U9: BMM150, Package_CSP:WLCSP-12_1.56x1.56mm_P0.4mm, symbol Sensor_Magnetic:BMM150
- added J5: JST SH 1.0, Connector_JST:JST_SH_SM04B-SRSS-TB_1x04-1MP_P1.00mm_Horizontal, symbol Connector_Generic_MountingPin:Conn_01x04_MountingPin
- added R38, R39: 10K, Resistor_SMD:R_0603_1608Metric, symbol Device:R
- added U4: LIS2MDL, Package_LGA:LGA-12_2x2mm_P0.5mm, symbol Sensor_Magnetic:LIS2MDL
- TP11: value PRDT -> INT
Connections:
- net +3V3: now also J5.3 (Pin_3), R38.1, U4.10 (Vdd_IO), U4.9 (Vdd); no longer C23.1
- net GND: now also J5.4 (Pin_4), R39.2, U4.6 (GND), U4.8 (GND)
- net SCL: now also J5.2 (Pin_2), U4.1 (SCL/SPC)
- net SDA: now also J5.1 (Pin_1), U4.4 (SDA/SDI/SDO)
- net at TP11.1: now also R39.1, U4.7 (DRDY)
- net ASCL: no longer names the net of U10.3 (ASCx)
- net ASDA: no longer names the net of U10.2 (ASDx)
- new net: R38.2, U4.3 (~{CS})
- new net: C23.1, U4.5 (C1)
- no-connect marks 3 -> 6
Other:
- note added: "LIS2MDL"
- note removed: "BMM150"
