File: DeltaT32.kicad_pcb (KiCad board)
At the start: 2 copper layers, 21.9 x 23.1 mm, 36 parts, among them J1 PH2.0, J2 USB_C_Receptacle_USB2.0_16P, J3 SH1.0, Q1 AO3401A, SW1 Boot, SW2 Reset, SW3 SW_SPDT_312, U1 TP4057, U2 MPU-6050, U3 ESP32-C3-MINI-1, U4 AP2112K-3.3

Commit message: Update Board
Parts:
- removed G***: LOGO, LOGO
- removed U4: AP2112K-3.3, Package_TO_SOT_SMD:SOT-23-5
- added C10: 1nF 10V, Capacitor_SMD:C_0402_1005Metric, F.Cu at (217.7, 97.0)
- added C11: DNP, Capacitor_SMD:C_0402_1005Metric, F.Cu at (202.8, 97.0)
- added C12: DNP, Capacitor_SMD:C_0402_1005Metric, F.Cu at (207.9, 97.0)
- added C18: 1uF 16V, Capacitor_SMD:C_0603_1608Metric, B.Cu at (128.6, 105.0)
- added C19: 2.2uF 16V, Capacitor_SMD:C_0603_1608Metric, B.Cu at (128.6, 102.5)
- added C20: 100nF 16V, Capacitor_SMD:C_0603_1608Metric, B.Cu at (128.6, 100.0)
- added C21: 100nF 16V, Capacitor_SMD:C_0603_1608Metric, B.Cu at (128.6, 97.5)
- added C22: 100nF 16V, Capacitor_SMD:C_0603_1608Metric, B.Cu at (128.6, 94.9)
- added C23: 100nF 16V, Capacitor_SMD:C_0603_1608Metric, B.Cu at (128.6, 92.4)
- added D5: LESD5D5.0CT1G, Diode_SMD:D_SOD-523, F.Cu at (214.1, 104.0)
- added D6: LESD5D5.0CT1G, Diode_SMD:D_SOD-523, F.Cu at (214.1, 105.7)
- added D7: B5819W, Diode_SMD:D_SOD-123, F.Cu at (212.4, 108.3)
- added D8: LESD5D5.0CT1G, Diode_SMD:D_SOD-523, F.Cu at (214.1, 102.3)
- added D9: B5819W, Diode_SMD:D_SOD-123, F.Cu at (204.8, 101.9)
- added J4: JST SH 1.0, Connector_JST:JST_SH_SM04B-SRSS-TB_1x04-1MP_P1.00mm_Horizontal, F.Cu at (166.1, 112.6)
- added JP1: SolderJumper_3_Bridged12, Jumper:SolderJumper-3_P1.3mm_Bridged2Bar12_RoundedPad1.0x1.5mm, B.Cu at (180.8, 89.9)
- added JP2: SolderJumper_3_Bridged12, Jumper:SolderJumper-3_P1.3mm_Bridged2Bar12_RoundedPad1.0x1.5mm, B.Cu at (180.9, 87.0)
- added L1: 2.2uH 2.2A, Inductor_SMD:L_Bourns-SRN4018, F.Cu at (202.1, 107.0)
- added Q4: BSS138, Package_TO_SOT_SMD:SOT-23, F.Cu at (174.9, 103.6)
- added Q5: BSS138, Package_TO_SOT_SMD:SOT-23, F.Cu at (179.1, 103.5)
- added R14: 10K, Resistor_SMD:R_0402_1005Metric, F.Cu at (198.8, 86.5)
- added R15: 1K, Resistor_SMD:R_0402_1005Metric, F.Cu at (205.4, 98.7)
- added R16: 442K, Resistor_SMD:R_0805_2012Metric, F.Cu at (212.0, 97.0)
- added R17: 160K, Resistor_SMD:R_0805_2012Metric, F.Cu at (215.4, 97.0)
- added R25: 10K, Resistor_SMD:R_0603_1608Metric, B.Cu at (132.6, 105.0)
- added R26: 10K, Resistor_SMD:R_0603_1608Metric, B.Cu at (132.6, 102.5)
- added R27: 10K, Resistor_SMD:R_0603_1608Metric, B.Cu at (132.6, 100.0)
- added R28: 10K, Resistor_SMD:R_0603_1608Metric, B.Cu at (132.6, 97.5)
- added R29: 0R, Resistor_SMD:R_0402_1005Metric, B.Cu at (132.9, 90.2)
- added R30: 10K, Resistor_SMD:R_0402_1005Metric, B.Cu at (132.9, 88.2)
- added R31: 10K, Resistor_SMD:R_0603_1608Metric, B.Cu at (132.6, 94.9)
- added R8: 0R, Resistor_SMD:R_0402_1005Metric, F.Cu at (221.8, 109.9)
- added R9: 100K, Resistor_SMD:R_0402_1005Metric, F.Cu at (195.4, 101.3)
- added TP1: TX, TestPoint:TestPoint_Pad_D1.0mm, B.Cu at (222.7, 86.6)
- added TP10: INT, TestPoint:TestPoint_Pad_D1.0mm, B.Cu at (174.9, 110.9)
- added TP11: PRDT, TestPoint:TestPoint_Pad_D1.0mm, B.Cu at (172.2, 110.8)
- added TP12: INT, TestPoint:TestPoint_Pad_D1.0mm, B.Cu at (175.3, 114.6)
- added TP2: RX, TestPoint:TestPoint_Pad_D1.0mm, B.Cu at (222.7, 88.6)
- added TP3: IO3, TestPoint:TestPoint_Pad_D1.0mm, B.Cu at (222.7, 94.6)
- added TP4: IO5, TestPoint:TestPoint_Pad_D1.0mm, B.Cu at (222.7, 92.6)
- added TP5: IO6, TestPoint:TestPoint_Pad_D1.0mm, B.Cu at (222.7, 90.6)
- added TP9: INT, TestPoint:TestPoint_Pad_D1.0mm, B.Cu at (172.3, 114.6)
- added U10: BMI160/270, Package_LGA:Bosch_LGA-14_3x2.5mm_P0.5mm, F.Cu at (170.7, 93.9)
- added U7: MAX30102, OptoDevice:Maxim_OLGA-14_3.3x5.6mm_P0.8mm, B.Cu at (169.8, 98.5)
- added U8: LN1134A182MR-G, Package_TO_SOT_SMD:SOT-23-5, F.Cu at (166.5, 105.6)
- added U9: BMM150, Package_CSP:WLCSP-12_1.56x1.56mm_P0.4mm, F.Cu at (171.3, 90.5)
- added Y1: 32.768Hz, Crystal:Crystal_SMD_3215-2Pin_3.2x1.5mm, F.Cu at (205.4, 97.0)
- added kibuzzard-61B9CE86: G***, label, F.Cu at (220.4, 95.6)
- added kibuzzard-61B9CEAB: G***, label, F.Cu at (220.4, 86.3)
- added kibuzzard-61B9EF98: G***, label_scaled_0.5, F.Cu at (213.2, 101.0)
- added kibuzzard-61C05335: G***, label, F.Cu at (205.0, 108.3)
- added kibuzzard-6269032F: G***, kibuzzard-6269032F, F.Cu at (200.2, 93.6)
- added kibuzzard-67F4DCFC: G***, kibuzzard-67F4DCFC, F.Cu at (212.5, 111.1)
- added kibuzzard-67F4DCFC: G***, kibuzzard-67F4DCFC, B.Cu at (212.5, 111.1)
- added kibuzzard-67F4DDA0: G***, kibuzzard-67F4DDA0, F.Cu at (214.4, 111.1)
- added kibuzzard-67F4DDA0: G***, kibuzzard-67F4DDA0, B.Cu at (214.5, 111.1)
- added kibuzzard-67F4E109: G***, kibuzzard-67F4E109, F.Cu at (201.6, 96.8)
- C1: value 1.0uF -> 10nF 10V; moved to F.Cu
- C2: value 10uF -> 100nF 10V; moved to F.Cu
- C3: value 10uF -> 1uF 16V; moved to F.Cu
- C4: value 100nF -> 1uF 16V; moved to F.Cu
- C5: value 2.2nF -> 4.7uF 16V; moved to F.Cu
- C6: value 100nF -> 4.7uF 16V; footprint Capacitor_SMD:C_0402_1005Metric -> Capacitor_SMD:C_0603_1608Metric; moved to F.Cu
- C7, C9: value 1.0uF -> 10uF 16V; footprint Capacitor_SMD:C_0402_1005Metric -> Capacitor_SMD:C_0805_2012Metric; moved to F.Cu
- C8: value 1.0uF -> 22pF 50V; footprint Capacitor_SMD:C_0402_1005Metric -> Capacitor_SMD:C_0603_1608Metric; moved to F.Cu
- D1: value RED -> LESD8D3.3CAT5G; footprint LED_SMD:LED_0402_1005Metric -> Diode_SMD:D_SOD-882
- D2: value BLUE -> WS2812B; footprint LED_SMD:LED_0402_1005Metric -> LED_SMD:LED_WS2812B-2020_PLCC4_2.0x2.0mm
- D3: value WS2812B-2020 -> BLUE LED; footprint LED_SMD:LED_WS2812B-2020_PLCC4_2.0x2.0mm -> LED_SMD:LED_0603_1608Metric
- D4: value MBR0530 -> RED LED; footprint Diode_SMD:D_SOD-123 -> LED_SMD:LED_0603_1608Metric
- J1: value PH2.0 -> JST SH 1.0; footprint Connector_JST:JST_PH_B2B-PH-SM4-TB_1x02-1MP_P2.00mm_Vertical -> Connector_JST:JST_SH_SM04B-SRSS-TB_1x04-1MP_P1.00mm_Horizontal; moved to F.Cu
- J2: value USB_C_Receptacle_USB2.0_16P -> JST PH 2.0; footprint Connector_USB:USB_C_Receptacle_GCT_USB4110 -> Connector_JST:JST_PH_B2B-PH-K_1x02_P2.00mm_Vertical
- J3: value SH1.0 -> USB C 16P; footprint Connector_JST:JST_SH_BM04B-SRSS-TB_1x04-1MP_P1.00mm_Vertical -> Connector_USB:USB_C_Receptacle_GCT_USB4105-xx-A_16P_TopMnt_Horizontal; moved to F.Cu
- Q1: value AO3401A -> DMG3415U; moved to F.Cu
- R1: value 10K -> 0R; moved to F.Cu
- R10: value 2K -> 22K1
- R11, R12: value 10K -> 5K1; moved to F.Cu
- R13: value 10K -> 100K; moved to F.Cu
- R2: value 2K -> 10K; moved to F.Cu
- R3: value 2K -> 10K
- R4: value 442K -> 0R; footprint Resistor_SMD:R_0805_2012Metric -> Resistor_SMD:R_0402_1005Metric; moved to F.Cu
- R5: value 160K -> 1K; footprint Resistor_SMD:R_0805_2012Metric -> Resistor_SMD:R_0402_1005Metric; moved to F.Cu
- R6: value 5.1K -> 470R; moved to F.Cu
- R7: value 5.1K -> 10K; moved to F.Cu
- SW1: value Boot -> MSK-12C02-07; footprint Button_Switch_SMD:SW_Push_SPST_NO_Alps_SKRK -> Button_Switch_SMD:SW_SPDT_PCM12
- SW2: value Reset -> BOOT; moved to F.Cu
- SW3: value SW_SPDT_312 -> RESET; footprint Button_Switch_SMD:SW_SPDT_PCM12 -> Button_Switch_SMD:SW_Push_SPST_NO_Alps_SKRK
- U1: value TP4057 -> ESP32-C3-MINI-1; footprint Package_TO_SOT_SMD:TSOT-23-6 -> PCM_Espressif:ESP32-C3-MINI-1; moved to F.Cu
- U2: value MPU-6050 -> MCP73831T-2ACI/OT; footprint Sensor_Motion:InvenSense_QFN-24_4x4mm_P0.5mm -> Package_TO_SOT_SMD:SOT-23-5; moved to F.Cu
- U3: value ESP32-C3-MINI-1 -> SY8088; footprint PCM_Espressif:ESP32-C3-MINI-1 -> Package_TO_SOT_SMD:SOT-23-5
- moved R12 113.7 mm to (219.8, 109.9), turned to 180 degrees
- moved J3 112.6 mm to (220.6, 103.9), turned to 90 degrees
- moved R11 110.7 mm to (221.8, 98.0)
- moved U2 106.3 mm to (208.2, 104.4), turned to 180 degrees
- moved D3 106.2 mm to (207.0, 108.3)
- moved J2 105.0 mm to (214.4, 113.4), turned to 180 degrees
- moved C6 104.8 mm to (211.0, 103.8), turned to -90 degrees
- moved R5 103.8 mm to (209.3, 107.4), turned to -90 degrees
- moved SW2 102.6 mm to (220.4, 89.0), turned to 0 degrees
- moved C5 100.7 mm to (205.3, 105.9), turned to 90 degrees
- moved J1 97.5 mm to (206.0, 112.8)
- moved R1 95.1 mm to (201.6, 94.4), turned to 90 degrees
- moved R6 94.7 mm to (213.0, 99.5)
- moved R13 94.5 mm to (209.0, 97.6)
- moved SW3 92.7 mm to (220.4, 93.0), turned to 0 degrees
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Connections:
- C1 pad 1: +3V3 -> +3.3V
- C2 pad 1: +BATT -> +3.3V
- C3 pad 1: VBUS -> +3.3V
- C4 pad 1: RESET -> CHIP_PU
- C5 pad 2: Net-(U2-REGOUT) -> VBUS
- C6 pad 1: Net-(U2-CPOUT) -> +BATT
- C7 pad 1: Net-(D4-K) -> +5V
- C8 pad 1: Net-(SW3-C) -> /Switch
- C8 pad 2: GND -> Net-(U3-FB)
- C9 pad 1: Net-(SW3-C) -> /Switch
- D1 pad 1: GND -> +3.3V
- D1 pad 2: Net-(D1-A) -> GND
- D2 pad 1: Net-(D2-K) -> +3.3V
- D2 pad 2: Net-(D2-A) -> unconnected-(D2-DOUT-Pad2)
- D3 pad 1: unconnected-(D3-DOUT-Pad1) -> Net-(D3-K)
- D3 pad 2: GND -> VBUS
- D4 pad 1: Net-(D4-K) -> GND
- D4 pad 2: VBUS -> Net-(D4-A)
- J1 pad 2: +BATT -> +3.3V
- J1 pad MP: GND -> unconnected-(J1-MountPin-PadMP)
- Q1 pad 2: Net-(D4-K) -> +5V
- R1 pad 1: BOOT -> IO3
- R1 pad 2: Net-(SW1-A) -> Net-(U1-GPIO3/ADC1_CH3)
- R10 pad 1: Net-(D2-A) -> Net-(U3-FB)
- R10 pad 2: VBUS -> GND
- R11 pad 1: +3V3 -> GND
- R11 pad 2: RESET -> Net-(J3-CC2)
- R12 pad 1: VBUS -> GND
- R12 pad 2: GND -> Net-(J3-CC1)
- R13 pad 1: Net-(D4-K) -> VBUS
- R13 pad 2: Net-(U4-EN) -> GND
- R2 pad 1: Net-(U1-PROG) -> +3.3V
- R2 pad 2: GND -> CHIP_PU
- R3 pad 1: +3V3 -> Net-(U2-PROG)
- R3 pad 2: Net-(D1-A) -> GND
- R4 pad 1: +BATT -> IO2
- R4 pad 2: SP_BAT -> Net-(D2-DIN)
- R5 pad 1: SP_BAT -> Net-(U2-STAT)
- R5 pad 2: GND -> Net-(D3-K)
- R6 pad 1: GND -> IO7
- R6 pad 2: Net-(J2-CC2) -> Net-(D4-A)
- R7 pad 1: GND -> +5V
- R7 pad 2: Net-(J2-CC1) -> EN
- SW1 pad 1: Net-(SW1-A) -> +3.3V
- SW1 pad 2: GND -> /Switch
- SW2 pad 1: RESET -> CHIP_PU
- SW3 pad 1: +3V3 -> BOOT
- SW3 pad 2: Net-(SW3-C) -> GND
- U1 pad 1: Net-(D2-K) -> GND
- U1 pad 3: +BATT -> +3.3V
- U1 pad 4: VBUS -> unconnected-(U1-NC-Pad4)
- U1 pad 5: unconnected-(U1-STDBY-Pad5) -> IO2
- U1 pad 6: Net-(U1-PROG) -> Net-(U1-GPIO3/ADC1_CH3)
- U2 pad 1: unconnected-(U2-CLKIN-Pad1) -> Net-(U2-STAT)
- U2 pad 2: unconnected-(U2-NC-Pad2) -> GND
- U2 pad 3: unconnected-(U2-NC-Pad3) -> +BATT
- U2 pad 4: unconnected-(U2-NC-Pad4) -> VBUS
- U2 pad 5: unconnected-(U2-NC-Pad5) -> Net-(U2-PROG)
- U3 pad 1: GND -> EN
- U3 pad 3: +3V3 -> /Buck_Coil
- U3 pad 4: unconnected-(U3-NC-Pad4) -> +5V
- U3 pad 5: unconnected-(U3-GPIO2/ADC1_CH2-Pad5) -> Net-(U3-FB)
Routing:
- net +3V3: track 70.2 -> 0.00 mm, vias 8 -> 0
- net GND: track 60.6 -> 12.1 mm, vias 19 -> 90
- net +3.3V: track 0.00 -> 44.6 mm, vias 0 -> 3
- net BOOT: track 4.96 -> 45.5 mm, vias 1 -> 5
- net Net-(U1-GPIO6): track 0.00 -> 27.6 mm, vias 0 -> 1
- net Net-(U1-GPIO5/ADC2_CH0): track 0.00 -> 27.3 mm, vias 0 -> 1
- net Net-(U1-GPIO4/ADC1_CH4): track 0.00 -> 27.1 mm, vias 0 -> 1
- net SCL: track 11.2 -> 37.8 mm, vias 1 -> 2
- net USB_D-: track 0.00 -> 24.2 mm, vias 0 -> 2
- net CHIP_PU: track 0.00 -> 22.4 mm, vias 0 -> 2
- net USB_D+: track 0.00 -> 21.5 mm, vias 0 -> 2
- net /Switch: track 0.00 -> 20.4 mm, vias 0 -> 2
- net SDA: track 10.5 -> 30.2 mm, vias 1 -> 2
- net IO3: track 0.00 -> 18.7 mm, vias 0 -> 2
- net Net-(SW3-C): track 17.5 -> 0.00 mm, vias 2 -> 0
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- added copper zone on F.Cu, net +5V
- added copper zone on B.Cu, net +BATT
- added copper zone on F.Cu, net +BATT
- added copper zone on F.Cu, net /Buck_Coil
- added copper zone on F.Cu, net /Switch
- added copper zone on B.Cu, net VBUS
Other:
- board size 21.9 x 23.1 mm -> 69.4 x 40.2 mm
- board text removed: "+-"
- board text removed: "0"
- board text removed: "C3-1"
- board text removed: "R"

Commit message: Update Board
Parts:
- removed C20: 100nF 16V, Capacitor_SMD:C_0603_1608Metric
- removed JP1, JP2: SolderJumper_3_Bridged12, Jumper:SolderJumper-3_P1.3mm_Bridged2Bar12_RoundedPad1.0x1.5mm
- removed TP12: INT, TestPoint:TestPoint_Pad_D1.0mm
- removed U9: BMM150, Package_CSP:WLCSP-12_1.56x1.56mm_P0.4mm
- removed kibuzzard-61B9CE86, kibuzzard-61B9CEAB, kibuzzard-61C05335: G***, label
- removed kibuzzard-61B9EF98: G***, label_scaled_0.5
- removed kibuzzard-67F4DCFC (x2): G***, kibuzzard-67F4DCFC
- removed kibuzzard-67F4DDA0 (x2): G***, kibuzzard-67F4DDA0
- added C24: 1uF 16V, Capacitor_SMD:C_0603_1608Metric, F.Cu at (198.0, 115.5)
- added C25: 2.2uF 16V, Capacitor_SMD:C_0603_1608Metric, F.Cu at (198.0, 111.8)
- added C26: 10nF 16V, Capacitor_SMD:C_0603_1608Metric, F.Cu at (198.0, 117.2)
- added C27: 100nF 16V, Capacitor_SMD:C_0603_1608Metric, F.Cu at (198.0, 113.7)
- added C28: 100nF 16V, Capacitor_SMD:C_0603_1608Metric, F.Cu at (201.8, 104.6)
- added J5: JST SH 1.0, Connector_JST:JST_SH_SM04B-SRSS-TB_1x04-1MP_P1.00mm_Horizontal, F.Cu at (227.9, 121.4)
- added Q6: BSS138, Package_TO_SOT_SMD:SOT-23, F.Cu at (197.7, 90.6)
- added Q7: BSS138, Package_TO_SOT_SMD:SOT-23, F.Cu at (201.8, 90.6)
- added R32: 10K, Resistor_SMD:R_0603_1608Metric, F.Cu at (199.5, 94.0)
- added R33: 10K, Resistor_SMD:R_0603_1608Metric, F.Cu at (197.8, 94.0)
- added R34: 10K, Resistor_SMD:R_0603_1608Metric, F.Cu at (200.5, 116.4)
- added R35: 10K, Resistor_SMD:R_0603_1608Metric, F.Cu at (202.4, 116.4)
- added R36: 0R, Resistor_SMD:R_0402_1005Metric, F.Cu at (204.6, 105.2)
- added R37: 10K, Resistor_SMD:R_0402_1005Metric, F.Cu at (203.3, 105.2)
- added R38: 10K, Resistor_SMD:R_0603_1608Metric, F.Cu at (234.8, 102.1)
- added R39: 10K, Resistor_SMD:R_0603_1608Metric, F.Cu at (231.2, 95.8)
- added TP13: INT, TestPoint:TestPoint_Pad_D1.0mm, F.Cu at (203.7, 98.1)
- added TP14: FSYNC, TestPoint:TestPoint_Pad_D1.0mm, F.Cu at (203.7, 102.1)
- added TP15: INT, TestPoint:TestPoint_Pad_D1.0mm, F.Cu at (203.7, 100.1)
- added U11: MAX30102, OptoDevice:Maxim_OLGA-14_3.3x5.6mm_P0.8mm, B.Cu at (197.7, 102.4)
- added U12: LN1134A182MR-G, Package_TO_SOT_SMD:SOT-23-5, F.Cu at (198.6, 109.0)
- added U13: MPU-9250, Sensor_Motion:InvenSense_QFN-24_3x3mm_P0.4mm_NoMask, F.Cu at (203.1, 109.3)
- added U4: LIS2MDL, Package_LGA:LGA-12_2x2mm_P0.5mm, F.Cu at (233.4, 97.0)
- C18, C19, C21, C22, C23, R25, R26, R27, R28, R29, R30, R31, TP10, TP9: moved to F.Cu
- J2: footprint Connector_JST:JST_PH_B2B-PH-K_1x02_P2.00mm_Vertical -> Connector_JST:JST_PH_S2B-PH-K_1x02_P2.00mm_Horizontal; moved to B.Cu
- TP11: value PRDT -> INT; moved to F.Cu
- moved C23 105.4 mm to (234.0, 94.1), turned to 180 degrees
- moved R29 105.3 mm to (236.7, 108.0), turned to 90 degrees
- moved R30 105.1 mm to (237.0, 102.4), turned to 90 degrees
- moved R28 105.0 mm to (236.2, 114.7), turned to 90 degrees
- moved C22 104.8 mm to (231.4, 115.5), turned to 180 degrees
- moved C21 104.7 mm to (231.4, 117.2), turned to 180 degrees
- moved C18 103.2 mm to (231.4, 113.7), turned to 180 degrees
- moved R27 102.8 mm to (234.4, 114.7), turned to 90 degrees
- moved R31 102.6 mm to (234.3, 108.5), turned to 90 degrees
- moved R25 102.4 mm to (234.1, 91.2)
- moved C19 102.2 mm to (230.7, 107.5)
- moved R26 98.1 mm to (230.0, 91.2), turned to 180 degrees
- moved TP9 69.0 mm to (237.2, 91.0)
- moved TP11 67.3 mm to (237.2, 93.0), turned to 0 degrees
- moved U10 65.6 mm to (235.4, 105.1)
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Connections:
- C23 pad 1: VDDIO -> Net-(U4-C1)
- J4 pad 1: GND -> SDA
- J4 pad 2: VDDIO -> SCL
- J4 pad 3: SCL -> VDDIO
- J4 pad 4: SDA -> GND
- U10 pad 2: ASDA -> unconnected-(U10-ASDx-Pad2)
- U10 pad 3: ASCL -> unconnected-(U10-ASCx-Pad3)
Routing:
- net SCL: track 37.8 -> 141.7 mm, vias 2 -> 9
- net VDDIO: track 4.27 -> 104.3 mm, vias 0 -> 5
- net SDA: track 30.2 -> 123.5 mm, vias 2 -> 9
- net +1V8: track 3.07 -> 70.6 mm, vias 0 -> 12
- net SCL_1V8: track 0.00 -> 46.7 mm, vias 0 -> 4
- net SDA_1V8: track 0.00 -> 43.8 mm, vias 0 -> 2
- net GND: track 12.1 -> 47.0 mm, vias 90 -> 78
- net Net-(U7-~{INT}): track 0.00 -> 16.7 mm, vias 0 -> 3
- net AD0: track 0.00 -> 11.4 mm, vias 0 -> 2
- net Net-(U10-INT1): track 0.00 -> 11.4 mm
- net Net-(U13-INT): track 0.00 -> 10.7 mm, vias 0 -> 2
- net Net-(U11-~{INT}): track 0.00 -> 10.1 mm, vias 0 -> 1
- net Net-(U4-DRDY): track 0.00 -> 9.12 mm, vias 0 -> 2
- net Net-(U13-FSYNC): track 0.00 -> 7.29 mm, vias 0 -> 2
- net Net-(U4-~{CS}): track 0.00 -> 6.48 mm
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- added copper zone on B.Cu, net +1V8
Other:
- board size 69.4 x 40.2 mm -> 99.4 x 44.5 mm

Commit message: Update Board
Parts:
- added G***: LOGO, LOGO, F.Cu at (165.3, 115.3)
- added kibuzzard-61C05335: G***, label, F.Cu at (155.6, 115.6)
- added kibuzzard-67FF2A33: G***, kibuzzard-67FF2A33, F.Cu at (155.7, 100.0)
- J1, TP10, TP11, TP9: moved to B.Cu
- moved R17 15.6 mm to (147.6, 107.8), turned to -90 degrees
- moved C19 11.3 mm to (229.9, 96.3), turned to -90 degrees
- moved U4 8.70 mm to (234.0, 105.7), turned to 90 degrees
- moved R16 8.56 mm to (153.2, 106.9), turned to 180 degrees
- moved R31 7.40 mm to (233.4, 115.8)
- moved R38 6.56 mm to (230.9, 107.4)
- moved C9 5.63 mm to (144.2, 115.6)
- moved L1 5.63 mm to (147.8, 115.0)
- moved D3 5.33 mm to (156.2, 114.3)
- moved R13 5.20 mm to (150.6, 103.5), turned to 180 degrees
- moved U10 4.86 mm to (235.6, 110.0), turned to -90 degrees
- moved U3 4.80 mm to (144.5, 110.2)
- moved U2 4.77 mm to (152.6, 111.4)
- moved R3 4.77 mm to (151.9, 113.8)
- moved R5 4.77 mm to (153.7, 114.4)
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Routing:
- net SCL: track 141.7 -> 163.1 mm, vias 9 -> 10
- net GND: track 47.0 -> 65.0 mm, vias 78 -> 93
- net +3.3V: track 44.6 -> 60.3 mm, vias 3 -> 4
- net VBUS: track 15.9 -> 30.6 mm, vias 6 -> 10
- net +BATT: track 5.48 -> 19.9 mm, vias 4 -> 3
- net +5V: track 11.2 -> 0.00 mm, vias 2 -> 0
- net SCL_1V8: track 46.7 -> 56.3 mm, vias 4 -> 6
- net VDDIO: track 104.3 -> 96.8 mm, vias 5 -> 2
- net Net-(U4-C1): track 2.66 -> 9.87 mm, vias 0 -> 2
- net /Switch: track 20.4 -> 26.6 mm, vias 2 -> 0
- net Net-(U10-CSB): track 1.80 -> 7.70 mm
- net Net-(U4-DRDY): track 9.12 -> 15.0 mm
- net +1V8: track 70.6 -> 76.2 mm, vias 12 -> 6
- net SDA: track 123.5 -> 128.7 mm, vias 9 -> 8
- net SDA_1V8: track 43.8 -> 39.6 mm, vias 2 -> 4
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- removed copper zone on B.Cu, net +BATT
