File: 340/Caps32Project.kicad_sch (KiCad schematic)
At the start: 37 parts, among them J1 Ph 2.0, J2 Sh 1.0, J4 Sh 2.0, P1 USB_C_Plug_USB2.0, Q1 AO3401A, Q2 MBT3904DW1, SW1 Reset, SW2 Boot, U1 MPU-6050, U2 MAX17048G_T10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

Commit message: Sync from 340 to main/340
Other:
- moved on the sheet: C6, D3
Changed lines of the file:
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@@
 	)
 	(no_connect
-		(at 201.93 127)
+		(at 177.8 90.17)
 	)
 	(no_connect
@@
 	(wire
 		(pts
+			(xy 185.42 81.28) (xy 185.42 82.55)
+		)
+		(stroke
+			(width 0)
+			(type default)
+		)
+	)
+	(wire
+		(pts
 			(xy 74.93 26.67) (xy 74.93 31.75)
 		)
@@
 	(wire
 		(pts
-			(xy 196.85 132.08) (xy 196.85 138.43)
+			(xy 172.72 95.25) (xy 172.72 101.6)
 		)
 		(stroke
@@
 	(wire
 		(pts
-			(xy 209.55 134.62) (xy 209.55 138.43)
+			(xy 185.42 97.79) (xy 185.42 101.6)
 		)
 		(stroke
@@
 	(wire
 		(pts
-			(xy 196.85 119.38) (xy 196.85 124.46)
+			(xy 172.72 81.28) (xy 172.72 87.63)
 		)
 		(stroke
@@
 	(global_label "RGB_DI"
 		(shape input)
-		(at 217.17 127 0)
+		(at 193.04 90.17 0)
 		(fields_autoplaced yes)
 		(effects
@@
 		)
 		(property "Intersheetrefs" "${INTERSHEET_REFS}"
-			(at 226.8076 127 0)
+			(at 202.6776 90.17 0)
 			(effects
 				(font
@@
 	(symbol
 		(lib_id "power:GND")
-		(at 196.85 138.43 0)
+		(at 172.72 101.6 0)
 		(unit 1)
 		(exclude_from_sim no)
@@
 		(fields_autoplaced yes)
 		(property "Reference" "#PWR037"
-			(at 196.85 144.78 0)
+			(at 172.72 107.95 0)
 			(effects
 				(font
@@
 		)
 		(property "Value" "GND"
-			(at 196.85 143.51 0)
+			(at 172.72 106.68 0)
 			(effects
 				(font
@@
 		)
 		(property "Footprint" ""
-			(at 196.85 138.43 0)
+			(at 172.72 101.6 0)
 			(effects
 				(font
@@
 		)
 		(property "Datasheet" ""
-			(at 196.85 138.43 0)
+			(at 172.72 101.6 0)
 			(effects
 				(font
@@
 		)
 		(property "Description" "Power symbol creates a global label with name \"GND\" , ground"
-			(at 196.85 138.43 0)
+			(at 172.72 101.6 0)
 			(effects
 				(font
@@
 	(symbol
 		(lib_id "power:+3V3")
-		(at 196.85 119.38 0)
+		(at 172.72 81.28 0)
 		(mirror y)
 		(unit 1)
@@
 		(fields_autoplaced yes)
 		(property "Reference" "#PWR036"
-			(at 196.85 123.19 0)
+			(at 172.72 85.09 0)
 			(effects
 				(font
@@
 		)
 		(property "Value" "+3V3"
-			(at 196.85 114.3 0)
+			(at 172.72 76.2 0)
 			(effects
 				(font
@@
 		)
 		(property "Footprint" ""
-			(at 196.85 119.38 0)
+			(at 172.72 81.28 0)
 			(effects
 				(font
@@
 		)
 		(property "Datasheet" ""
-			(at 196.85 119.38 0)
+			(at 172.72 81.28 0)
 			(effects
 				(font
@@
 		)
 		(property "Description" "Power symbol creates a global label with name \"+3V3\""
-			(at 196.85 119.38 0)
+			(at 172.72 81.28 0)
 			(effects
 				(font
@@
 	(symbol
 		(lib_id "LED:WS2812B")
-		(at 209.55 127 0)
+		(at 185.42 90.17 0)
 		(mirror y)
 		(unit 1)
@@
 		(dnp no)
 		(property "Reference" "D3"
-			(at 207.01 120.142 0)
+			(at 182.88 83.312 0)
 			(effects
 				(font
@@
 		)
 		(property "Value" "WS2812B"
-			(at 198.12 123.2214 0)
+			(at 173.99 86.3914 0)
 			(effects
 				(font
@@
 		)
 		(property "Footprint" "LED_SMD:LED_WS2812B_PLCC4_5.0x5.0mm_P3.2mm"
-			(at 208.28 134.62 0)
+			(at 184.15 97.79 0)
 			(effects
 				(font
@@
 		)
 		(property "Datasheet" "https://cdn-shop.adafruit.com/datasheets/WS2812B.pdf"
-			(at 207.01 136.525 0)
+			(at 182.88 99.695 0)
 			(effects
 				(font
@@
 		)
 		(property "Description" "RGB LED with integrated controller"
-			(at 209.55 127 0)
+			(at 185.42 90.17 0)
 			(effects
 				(font
@@
 	(symbol
 		(lib_id "power:GND")
-		(at 209.55 138.43 0)
+		(at 185.42 101.6 0)
 		(mirror y)
 		(unit 1)
@@
 		(fields_autoplaced yes)
 		(property "Reference" "#PWR021"
-			(at 209.55 144.78 0)
+			(at 185.42 107.95 0)
 			(effects
 				(font
@@
 		)
 		(property "Value" "GND"
-			(at 209.55 143.51 0)
+			(at 185.42 106.68 0)
 			(effects
 				(font
@@
 		)
 		(property "Footprint" ""
-			(at 209.55 138.43 0)
+			(at 185.42 101.6 0)
 			(effects
 				(font
@@
 		)
 		(property "Datasheet" ""
-			(at 209.55 138.43 0)
+			(at 185.42 101.6 0)
 			(effects
 				(font
@@
 		)
 		(property "Description" "Power symbol creates a global label with name \"GND\" , ground"
-			(at 209.55 138.43 0)
+			(at 185.42 101.6 0)
 			(effects
 				(font
@@
 	(symbol
 		(lib_id "power:+3V3")
-		(at 209.55 119.38 0)
+		(at 185.42 81.28 0)
 		(unit 1)
 		(exclude_from_sim no)
@@
 		(fields_autoplaced yes)
 		(property "Reference" "#PWR035"
-			(at 209.55 123.19 0)
+			(at 185.42 85.09 0)
 			(effects
 				(font
@@
 		)
 		(property "Value" "+3V3"
-			(at 209.55 114.3 0)
+			(at 185.42 76.2 0)
 			(effects
 				(font
@@
 		)
 		(property "Footprint" ""
-			(at 209.55 119.38 0)
+			(at 185.42 81.28 0)
 			(effects
 				(font
@@
 		)
 		(property "Datasheet" ""
-			(at 209.55 119.38 0)
+			(at 185.42 81.28 0)
 			(effects
 				(font
@@
 		)
 		(property "Description" "Power symbol creates a global label with name \"+3V3\""
-			(at 209.55 119.38 0)
+			(at 185.42 81.28 0)
 			(effects
 				(font
@@
 	(symbol
 		(lib_id "Device:C")
-		(at 196.85 128.27 0)
+		(at 172.72 91.44 0)
 		(unit 1)
 		(exclude_from_sim no)
@@
 		(dnp no)
 		(property "Reference" "C6"
-			(at 196.85 126.238 0)
+			(at 172.72 89.408 0)
 			(effects
 				(font
@@
 		)
 		(property "Value" "1.0uF"
-			(at 197.104 130.81 0)
+			(at 172.974 93.98 0)
 			(effects
 				(font
@@
 		)
 		(property "Footprint" "Capacitor_SMD:C_0402_1005Metric_Pad0.74x0.62mm_HandSolder"
-			(at 197.8152 132.08 0)
+			(at 173.6852 95.25 0)
 			(effects
 				(font
@@
 		)
 		(property "Datasheet" "~"
-			(at 196.85 128.27 0)
+			(at 172.72 91.44 0)
 			(effects
 				(font
@@
 		)
 		(property "Description" "Unpolarized capacitor"
-			(at 196.85 128.27 0)
+			(at 172.72 91.44 0)
 			(effects
 				(font
