File: esp-unit-c3-v2/esp-unit-c3-v2.kicad_sch (KiCad schematic)
At the start: 55 parts, among them J1 JST SH 1.0, J2 JST PH 2.0, J3 USB C 16P, Q1 DMG3415U, SW1 MSK-12C02-07, SW2 BOOT, SW3 RESET, U1 ESP32-C3-MINI-1, U2 MCP73831T-2ACI/OT, U3 SY8088, Y1 32.768Hz

Commit message: Downgrade and pcb breakdown
Parts:
- removed D1: LESD8D3.3CAT5G, Diode_SMD:D_SOD-882, symbol Device:D_TVS
- removed D2: WS2812B, LED_SMD:LED_WS2812B-2020_PLCC4_2.0x2.0mm, symbol LED:WS2812B
- removed D5: LESD5D5.0CT1G, Diode_SMD:D_SOD-523, symbol Device:D_TVS
- removed D9: B5819W, Diode_SMD:D_SOD-123, symbol Device:D_Schottky
- removed L1: 2.2uH 2.2A, Inductor_SMD:L_Bourns-SRN4018, symbol Device:L
- removed SW1: MSK-12C02-07, Button_Switch_SMD:SW_SPDT_PCM12, symbol Switch:SW_SPDT_312
- removed SW3: RESET, Button_Switch_SMD:SW_Push_SPST_NO_Alps_SKRK, symbol Switch:SW_Push
- removed TP2: RX, TestPoint:TestPoint_Pad_D1.0mm, symbol Connector:TestPoint
- removed TP3: IO3, TestPoint:TestPoint_Pad_D1.0mm, symbol Connector:TestPoint
- removed TP4: IO5, TestPoint:TestPoint_Pad_D1.0mm, symbol Connector:TestPoint
- removed TP5: IO6, TestPoint:TestPoint_Pad_D1.0mm, symbol Connector:TestPoint
- removed U2: MCP73831T-2ACI/OT, Package_TO_SOT_SMD:SOT-23-5, symbol Battery_Management:MCP73831-2-OT
- removed U3: SY8088, Package_TO_SOT_SMD:SOT-23-5, symbol Rust_Board:SY8088
- added D1: WS2812B, LED_SMD:LED_WS2812B-2020_PLCC4_2.0x2.0mm, symbol LED:WS2812B-2020
- added D2: LESD8D3.3CAT5G, Diode_SMD:D_SOD-882, symbol Device:D_TVS
- added D5: B5819W, Diode_SMD:D_SOD-123, symbol Device:D_Schottky
- added D9: LESD5D5.0CT1G, Diode_SMD:D_SOD-523, symbol Device:D_TVS
- added L1: SPH4018H2R2MT (2.2uH 2.2A), Inductor_SMD:L_Bourns-SRN4018, symbol Device:L_Small
- added R18: 160K, Resistor_SMD:R_0805_2012Metric, symbol Device:R
- added R19, R20: 0R, Resistor_SMD:R_0402_1005Metric, symbol Device:R
- added SW1: BOOT, Button_Switch_SMD:SW_Push_SPST_NO_Alps_SKRK, symbol Switch:SW_Push
- added SW3: MSK-12C02-07, Button_Switch_SMD:SW_SPDT_PCM12, symbol Switch:SW_SPDT_312
- added U2: Delta_Board-1, DeltaT32:Delta_Board-1, symbol Rust_Board:Rust_Board
- added U3: MCP73831T-2ACI/OT, Package_TO_SOT_SMD:SOT-23-5, symbol Battery_Management:MCP73831-2-OT
- added U4: SY8088, Package_TO_SOT_SMD:SOT-23-5, symbol Rust_Board:SY8088
- C10: value 1nF 10V -> 10uF 16V; footprint Capacitor_SMD:C_0402_1005Metric -> Capacitor_SMD:C_0805_2012Metric; LCSC C1523 -> C15850; now in the parts list
- C11: value DNP -> 22pF 50V; footprint Capacitor_SMD:C_0402_1005Metric -> Capacitor_SMD:C_0603_1608Metric; LCSC (none) -> C1653; now in the parts list
- C12: value DNP -> 10uF 16V; footprint Capacitor_SMD:C_0402_1005Metric -> Capacitor_SMD:C_0805_2012Metric; LCSC (none) -> C15850; now in the parts list
- C5, C6: value 4.7uF 16V -> DNP; footprint Capacitor_SMD:C_0603_1608Metric -> Capacitor_SMD:C_0402_1005Metric; LCSC C19666 -> (none); now left out of the parts list
- C7, C9: value 10uF 16V -> 4.7uF 16V; footprint Capacitor_SMD:C_0805_2012Metric -> Capacitor_SMD:C_0603_1608Metric; LCSC C15850 -> C19666
- C8: value 22pF 50V -> 1nF 10V; footprint Capacitor_SMD:C_0603_1608Metric -> Capacitor_SMD:C_0402_1005Metric; LCSC C1653 -> C1523; now left out of the parts list
- D3: LCSC (none) -> C2286
- J1: value JST SH 1.0 -> JST SH1.0
- J2: value JST PH 2.0 -> JST PH2.0
- R1: LCSC (none) -> C17168
- R10: value 22K1 -> 100K; LCSC (none) -> C25741
- R11: value 5K1 -> 0R; LCSC (none) -> C17168
- R12: value 5K1 -> 10K; LCSC (none) -> C25744
- R13: value 100K -> 5K1; LCSC (none) -> C25905
- R14: value 10K -> 5K1; LCSC (none) -> C25905
- R15: value 1K -> 100K; LCSC (none) -> C25741
- R16: value 442K -> 22K1; footprint Resistor_SMD:R_0805_2012Metric -> Resistor_SMD:R_0402_1005Metric; LCSC (none) -> C43473
- R17: value 160K -> 442K
- R2, R7: LCSC (none) -> C25744
- R3: value 10K -> 470R; LCSC (none) -> C25117
- R4, R8: value 0R -> 10K; LCSC (none) -> C25744
- R5: value 1K -> 10K; LCSC (none) -> C25744
- R6: value 470R -> DNP
- R9: value 100K -> 1K; LCSC (none) -> C11702
- SW2: value BOOT -> RESET
- TP1: value TX -> ENABLE; now in the parts list
Connections:
- net +5V: now also C10.1, R12.2, D5.1 (K), U4.4 (IN); no longer C7.1, R7.1
- net +BATT: now also C9.1, R17.2, U3.3 (VBAT); no longer C6.1, R16.1
- net Buck_Coil: now also L1.1, U4.3 (LX)
- net CHIP_PU: now also R5.2; no longer R2.2
- net GND: now also C1.1, C10.2, C2.1, C3.1, C5.2, C7.1, C8.2, D3.1 (K), R10.1, R13.1, R14.1, R16.1, R7.1, D1.2 (VSS), D2.1 (A1), D9.2 (A2), R18.1, SW1.2, U2.2 (GND), U3.2 (VSS), U4.2 (GND); no longer C1.2, C10.1, C11.2, C2.2, C3.2, C5.1, C7.2, D4.1 (K), R10.2, R12.1, R13.2, R17.2, R3.2, R8.1
- net IO0: now also C5.1, R6.1; no longer C11.1, R15.1
- net IO1: now also C6.1, R6.2; no longer C12.1, R15.2
- net IO2: now also R1.1, U2.5 (A2/GPIO2); no longer R4.1
- net IO3: now also U1.6 (GPIO3/ADC1_CH3), R19.1, U2.6 (A3/GPIO3); no longer R1.1, R16.2, R17.1
- net IO7: now also R3.1, U2.10 (GPIO7); no longer R6.1
- net Switch: now also C11.1, C12.1, R15.2, L1.2, SW3.2 (C); no longer C8.1, C9.1, R9.1
- net USB_D+: now also D6.1 (A1)
- net USB_D-: now also D9.1 (A1); no longer D6.1 (A1)
- net VBUS: now also C7.2, D4.2 (A), R10.2, D5.2 (A), U3.4 (VDD); no longer C5.2, D3.2 (A), R13.1
- net IO4: now reaches U1.18 (GPIO4/ADC1_CH4)
- net IO4: now also R20.1, U2.7 (A4/GPIO4)
- net +3V3: now reaches R5.1
- net +3V3: now also C1.2, C2.2, C3.2, J1.2 (Pin_2), R2.2, R4.2, R8.2, U1.3 (3V3), D1.4 (VDD), D2.2 (A2), SW3.1 (B), U2.1 (3V3)
- net IO5: now reaches U1.19 (GPIO5/ADC2_CH0)
- net IO5: now also U2.8 (A5/GPIO5)
- net IO6: now reaches U1.20 (GPIO6)
- net IO6: now also U2.9 (GPIO6)
- net IO20_RX: now reaches U1.30 (GPIO20/U0RXD)
- net IO20_RX: now also U2.11 (RXD/GPIO20)
- net at TP1.1: now also R12.1, R20.2, U4.1 (EN); no longer U1.31 (GPIO21/U0TXD)
- net at R1.2: now also D1.3 (DIN); no longer U1.6 (GPIO3/ADC1_CH3)
- net at J3.B5 (CC2): now also R14.2; no longer R11.2
- net at J3.S1 (SHIELD): now also R11.2; no longer R8.2
- net at J3.A5 (CC1): now also R13.2; no longer R12.2
- removed net +3.3V: C1.1, C2.1, C3.1, J1.2 (Pin_2), R14.1, R2.1, U1.3 (3V3)
- removed net BOOT: C10.2, R14.2, U1.23 (GPIO9)
- net EN: no longer names the net of R7.2
- net EN: now also U3.5 (PROG)
- net SCL renamed IO10_SDA
- net IO10_SDA: now also R2.1, U1.16 (GPIO10), U2.4 (SDA/GPIO10); no longer U1.22 (GPIO8)
- net SDA renamed IO8_SCL
- net IO8_SCL: now also R4.1, U1.22 (GPIO8), U2.3 (SCL/GPIO8); no longer U1.16 (GPIO10)
- new net: R17.1, R18.2, R19.2
- new net: C11.2, R15.1, R16.2, U4.5 (FB)
- new net: R9.1, U3.1 (STAT)
- new net: D4.1 (K), R9.2
- new net: D3.2 (A), R3.2
- new net IO21_TX: U1.31 (GPIO21/U0TXD), U2.12 (TXD/GPIO21)
- new net IO9_BOOT: C8.1, R8.1, SW1.1, U1.23 (GPIO9)
Other:
- removed sheet BMI
- removed sheet MPU9250
- note added: "DEV BOARD"
- note added: "ESP32-C3-MINI-1"
- note added: "JST Connector (SH1.0 & PH2.0)"
- note added: "V.BAT"
- note removed: "ESP32-C3-MINI-1 Module"
- note removed: "IMU & Heart Rate Sensor"
- note removed: "IMU Default : 0x68 (1101000b) Alternative : 0x69 (1101001b) Heart-Rate Sensor Default : 0x57 (1010111b)"
- note removed: "Voltage Divider"
- title: DeltaT32 -> esp-unit-c3-v2

Commit message: add sensor board
Parts:
- J2: footprint Connector_JST:JST_PH_S2B-PH-K_1x02_P2.00mm_Horizontal -> DeltaT32:JST_PH2.0
- SW3: footprint Button_Switch_SMD:SW_SPDT_PCM12 -> DeltaT32:MSK-12C02-07
Changed lines of the file:
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@@
 			)
 		)
-		(property "Footprint" "Connector_JST:JST_PH_S2B-PH-K_1x02_P2.00mm_Horizontal"
+		(property "Footprint" "DeltaT32:JST_PH2.0"
 			(at 96.52 120.65 0)
 			(effects
@@
 			)
 		)
-		(property "Footprint" "Button_Switch_SMD:SW_SPDT_PCM12"
+		(property "Footprint" "DeltaT32:MSK-12C02-07"
 			(at 257.81 39.37 0)
 			(effects
