File: sensor-bmi/sensor-bmi.kicad_sch (KiCad schematic)
At the start: 24 parts, among them J5 JST SH 1.0, Q4 BSS138, Q5 BSS138, U10 BMI160/270, U4 LIS2MDL, U7 MAX30102, U8 LN1134A182MR-G

Commit message: Downgrade and pcb breakdown
Parts:
- removed C18: 1uF 16V, Capacitor_SMD:C_0603_1608Metric, symbol Device:C_Small
- removed C19: 2.2uF 16V, Capacitor_SMD:C_0603_1608Metric, symbol Device:C_Small
- removed C21, C22, C23: 100nF 16V, Capacitor_SMD:C_0603_1608Metric, symbol Device:C_Small
- removed J5: JST SH 1.0, Connector_JST:JST_SH_SM04B-SRSS-TB_1x04-1MP_P1.00mm_Horizontal, symbol Connector_Generic_MountingPin:Conn_01x04_MountingPin
- removed Q4, Q5: BSS138, Package_TO_SOT_SMD:SOT-23, symbol Transistor_FET:BSS138
- removed R25, R26, R27, R28, R31, R38, R39: 10K, Resistor_SMD:R_0603_1608Metric, symbol Device:R
- removed R29: 0R, Resistor_SMD:R_0402_1005Metric, symbol Device:R
- removed R30: 10K, Resistor_SMD:R_0402_1005Metric, symbol Device:R
- removed TP10, TP11, TP9: INT, TestPoint:TestPoint_Pad_D1.0mm, symbol Connector:TestPoint
- removed U10: BMI160/270, Package_LGA:Bosch_LGA-14_3x2.5mm_P0.5mm, symbol Sensor_Motion:BMI160
- removed U4: LIS2MDL, Package_LGA:LGA-12_2x2mm_P0.5mm, symbol Sensor_Magnetic:LIS2MDL
- removed U7: MAX30102, OptoDevice:Maxim_OLGA-14_3.3x5.6mm_P0.8mm, symbol Sensor:MAX30102
- removed U8: LN1134A182MR-G, Package_TO_SOT_SMD:SOT-23-5, symbol Regulator_Linear:AP2112K-1.8
- added C1: 1uF 16V, Capacitor_SMD:C_0603_1608Metric, symbol Device:C_Small
- added C2: 2.2uF 16V, Capacitor_SMD:C_0603_1608Metric, symbol Device:C_Small
- added C3, C4, C5: 100nF 16V, Capacitor_SMD:C_0603_1608Metric, symbol Device:C_Small
- added J1: JST SH1.0, Connector_JST:JST_SH_SM04B-SRSS-TB_1x04-1MP_P1.00mm_Horizontal, symbol Connector_Generic_MountingPin:Conn_01x04_MountingPin
- added Q1, Q2: BSS138, Package_TO_SOT_SMD:SOT-23, symbol Transistor_FET:BSS138
- added R1, R2, R3, R4, R5, R6, R8, R9: 10K, Resistor_SMD:R_0402_1005Metric, symbol Device:R
- added R7: 0R, Resistor_SMD:R_0402_1005Metric, symbol Device:R
- added TP1: MAX_INT, TestPoint:TestPoint_Pad_D1.0mm, symbol Connector:TestPoint
- added TP2: LIS_INT, TestPoint:TestPoint_Pad_D1.0mm, symbol Connector:TestPoint
- added TP3: BMI_INT, TestPoint:TestPoint_Pad_D1.0mm, symbol Connector:TestPoint
- added U1: LN1134A182MR-G, Package_TO_SOT_SMD:SOT-23-5, symbol Regulator_Linear:AP2112K-3.3
- added U2: MAX30102, OptoDevice:Maxim_OLGA-14_3.3x5.6mm_P0.8mm, symbol Sensor:MAX30102
- added U3: LIS2MDL, Package_LGA:LGA-12_2x2mm_P0.5mm, symbol Sensor_Magnetic:LIS2MDL
- added U4: BMI160, Package_LGA:Bosch_LGA-14_3x2.5mm_P0.5mm, symbol Sensor_Motion:BMI160
Connections:
- net +1V8: now also Q1.1 (G), Q2.1 (G), R1.1, R2.1, U2.11 (VDD)
- net +3V3: now also C1.1, C2.1, C4.1, C5.1, J1.3 (Pin_3), R3.1, R4.2, R5.2, R7.1, R9.1, U1.1 (VIN), U1.3 (EN), U1.5 (VOUT), U2.10 (VLED+), U2.9 (VLED+), U3.10 (Vdd_IO), U3.9 (Vdd), U4.5 (VDDIO), U4.8 (VDD)
- net GND: now also C1.2, C2.2, C3.2, C4.2, C5.2, J1.4 (Pin_4), R6.2, R8.2, U1.2 (GND), U2.12 (GND), U2.4 (PGND), U3.6 (GND), U3.8 (GND), U4.6 (GNDIO), U4.7 (GND)
- net SCL: now also J1.2 (Pin_2), Q1.3 (D), R5.1, U3.1 (SCL/SPC), U4.13 (SCx)
- net SCL_1V8: now also Q1.2 (S), R2.2, U2.2 (SCL)
- net SDA: now also J1.1 (Pin_1), Q2.3 (D), R4.1, U3.4 (SDA/SDI/SDO), U4.14 (SDx)
- net SDA_1V8: now also Q2.2 (S), R1.2, U2.3 (SDA)
- new net: R3.2, U3.3 (~{CS})
- new net: R6.1, TP2.1, U3.7 (DRDY)
- new net: R7.2, R8.1, U4.1 (SDO)
- new net: R9.2, U4.12 (CSB)
- new net: TP3.1, U4.4 (INT1)
- new net: TP1.1, U2.13 (~{INT})
- new net: C3.1, U3.5 (C1)
Other:
- note added: "JST Port"
- title: (none) -> sensor-unit-bmi

Commit message: add sensor board
Connections:
- net +1V8: now also C2.1, U1.5 (VOUT)
- net +3V3: no longer C2.1, U1.5 (VOUT)
Changed lines of the file:
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@@
+	)
+	(symbol
+		(lib_id "power:+1V8")
+		(at 49.53 30.48 0)
+		(unit 1)
+		(exclude_from_sim no)
+		(in_bom yes)
+		(on_board yes)
+		(dnp no)
+		(fields_autoplaced yes)
+		(property "Reference" "#PWR05"
+			(at 49.53 34.29 0)
+			(effects
+				(font
+					(size 1.27 1.27)
+				)
+				(hide yes)
+			)
+		)
+		(property "Value" "+1V8"
+			(at 49.53 25.4 0)
+			(effects
+				(font
+					(size 1.27 1.27)
+				)
+			)
+		)
+		(property "Footprint" ""
+			(at 49.53 30.48 0)
+			(effects
+				(font
+					(size 1.27 1.27)
+				)
+				(hide yes)
+			)
+		)
+		(property "Datasheet" ""
+			(at 49.53 30.48 0)
+			(effects
+				(font
+					(size 1.27 1.27)
+				)
+				(hide yes)
+			)
+		)
+		(property "Description" "Power symbol creates a global label with name \"+1V8\""
+			(at 49.53 30.48 0)
+			(effects
+				(font
+					(size 1.27 1.27)
+				)
+				(hide yes)
+			)
+		)
+		(pin "1"
+		)
+		(instances
+			(project "sensor-bmi"
+				(path "/112ff685-7007-423e-a7bc-97a8d4f3e1a8"
+					(reference "#PWR05")
+					(unit 1)
+				)
+			)
+		)
 	)
 	(symbol
@@
 					(unit 1)
 				)
-			)
-		)
-	)
-	(symbol
-		(lib_id "power:+3V3")
-		(at 49.53 30.48 0)
-		(unit 1)
-		(exclude_from_sim no)
-		(in_bom yes)
-		(on_board yes)
-		(dnp no)
-		(fields_autoplaced yes)
-		(property "Reference" "#PWR05"
-			(at 49.53 34.29 0)
-			(effects
-				(font
-					(size 1.27 1.27)
-				)
-				(hide yes)
-			)
-		)
-		(property "Value" "+3V3"
-			(at 49.53 25.4 0)
-			(effects
-				(font
-					(size 1.27 1.27)
-				)
-			)
-		)
-		(property "Footprint" ""
-			(at 49.53 30.48 0)
-			(effects
-				(font
-					(size 1.27 1.27)
-				)
-				(hide yes)
-			)
-		)
-		(property "Datasheet" ""
-			(at 49.53 30.48 0)
-			(effects
-				(font
-					(size 1.27 1.27)
-				)
-				(hide yes)
-			)
-		)
-		(property "Description" "Power symbol creates a global label with name \"+3V3\""
-			(at 49.53 30.48 0)
-			(effects
-				(font
-					(size 1.27 1.27)
-				)
-				(hide yes)
-			)
-		)
-		(pin "1"
-		)
-		(instances
-			(project ""
-				(path "/112ff685-7007-423e-a7bc-97a8d4f3e1a8"
-					(reference "#PWR05")
-					(unit 1)
-				)
