File: sensor-bmi/sensor-bmi.kicad_pcb (KiCad board)
At the start: 2 copper layers, 31.2 x 42 mm, 32 parts, among them J1 JST SH1.0, Q1 BSS138, Q2 BSS138, U1 LN1134A182MR-G, U2 MAX30102, U3 LIS2MDL, U4 BMI160

Commit message: panelize sensor board
Parts:
- added kibuzzard-68103EF6: G***, kibuzzard-68103EF6, F.Cu at (174.8, 84.9)
- added kibuzzard-68103EF6: G***, kibuzzard-68103EF6, B.Cu at (174.8, 84.9)
- added mouse-bite-2mm-slot: VAL**, Panelization Pretty:mouse-bite-2mm-slot, F.Cu at (185.3, 90.9)
- added mouse-bite-2mm-slot: VAL**, Panelization Pretty:mouse-bite-2mm-slot, F.Cu at (185.3, 78.9)
- added mouse-bite-2mm-slot: VAL**, Panelization Pretty:mouse-bite-2mm-slot, F.Cu at (174.8, 101.9)
- moved R4 2.81 mm to (192.1, 103.9), turned to 0 degrees
Routing:
- net +3V3: track 38.7 -> 42.8 mm
- net SDA: track 59.8 -> 56.3 mm
- net GND: track 4.58 -> 5.97 mm, vias 30 -> 33
- net SCL_1V8: track 10.8 -> 9.56 mm
- net Net-(U3-DRDY): track 30.7 -> 31.4 mm
Other:
- outline, holes or cut-outs redrawn

Commit message: resizing pcb board
Other:
- board size 31.2 x 42 mm -> 167.1 x 65.4 mm
