File: esp-unit-c3-v3/esp-unit-c3-v3.kicad_pcb (KiCad board)
At the start: 2 copper layers, 40 x 40 mm, 86 parts, among them J1 Conn_01x04, J2 JST PH2.0, J3 USB C 16P, Q1 DMG3415U, SW1 BOOT, SW2 RESET, SW3 MSK-12C02-07, U1 ESP32-C3-MINI-1, U3 MCP73831T-2ACI/OT, U4 SY8088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

Commit message: Update board
Parts:
- added kibuzzard-680CFCF0: G***, kibuzzard-680CFCF0, B.Cu at (113.1, 76.5)
- added kibuzzard-680CFD12: G***, kibuzzard-680CFD12, B.Cu at (113.1, 79.0)
- added kibuzzard-680CFD73: G***, kibuzzard-680CFD73, B.Cu at (113.1, 86.7)
- added kibuzzard-680CFD7F: G***, kibuzzard-680CFD7F, B.Cu at (113.1, 89.3)
- added kibuzzard-680CFDA8: G***, kibuzzard-680CFDA8, B.Cu at (145.1, 74.2)
- added kibuzzard-680CFDBB: G***, kibuzzard-680CFDBB, B.Cu at (145.1, 76.7)
- added kibuzzard-680CFDCF: G***, kibuzzard-680CFDCF, B.Cu at (145.7, 86.9)
- added kibuzzard-680CFDE4: G***, kibuzzard-680CFDE4, B.Cu at (145.8, 89.4)
- added kibuzzard-680CFDFB: G***, kibuzzard-680CFDFB, B.Cu at (113.1, 94.3)
- added kibuzzard-680CFE08: G***, kibuzzard-680CFE08, B.Cu at (113.1, 91.8)
- added kibuzzard-6816DDEA: G***, kibuzzard-6816DDEA, B.Cu at (113.1, 81.6)
- added kibuzzard-6816DDFD: G***, kibuzzard-6816DDFD, B.Cu at (113.1, 84.2)
- added kibuzzard-6816DE5B: G***, kibuzzard-6816DE5B, B.Cu at (145.2, 84.4)
- added kibuzzard-6816DE78: G***, kibuzzard-6816DE78, B.Cu at (145.1, 79.2)
- added kibuzzard-6816DE97: G***, kibuzzard-6816DE97, B.Cu at (145.2, 81.8)
- added kibuzzard-6816EC1C: G***, kibuzzard-6816EC1C, F.Cu at (112.6, 74.0)
- added kibuzzard-6816EC1C: G***, kibuzzard-6816EC1C, B.Cu at (112.6, 74.0)
- U2: value ~ -> Delta Board 2
- moved R12 113.7 mm to (115.5, 95.7)
- moved R15 113.7 mm to (115.5, 91.8)
- moved R16 113.7 mm to (115.5, 93.7)
- moved SW3 113.7 mm to (120.2, 105.0)
- moved C1 113.7 mm to (119.6, 73.9)
- moved C10 113.7 mm to (121.0, 93.2)
- moved C2 113.7 mm to (120.6, 73.9)
- moved C4 113.7 mm to (121.7, 79.8)
- moved C5 113.7 mm to (122.2, 85.3)
- moved C7 113.7 mm to (123.9, 96.8)
- moved C9 113.7 mm to (131.1, 95.4)
- moved D1 113.7 mm to (116.9, 80.3)
- moved D3 113.7 mm to (116.9, 82.8)
- moved D4 113.7 mm to (126.6, 104.9)
- moved D5 113.7 mm to (123.9, 92.7)
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