File: esp-unit-c3-v3/esp-unit-c3-v3.kicad_sch (KiCad schematic)
At the start: 55 parts, among them J1 Conn_01x04, J2 JST PH2.0, J3 USB C 16P, Q1 DMG3415U, SW1 BOOT, SW2 RESET, SW3 MSK-12C02-07, U1 ESP32-C3-MINI-1, U3 MCP73831T-2ACI/OT, U4 SY8088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

Commit message: Update board
Parts:
- U2: value ~ -> Delta Board 2
Changed lines of the file:
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@@
 			)
 		)
-		(property "Value" "~"
+		(property "Value" "Delta Board 2"
 			(at 44.45 154.94 0)
 			(effects
