File: hardware/esp-unit-c3-v3/esp-unit-c3-v3.kicad_pcb (KiCad board)
At the start: 2 copper layers, 40 x 40 mm, 103 parts, among them J1 Conn_01x04, J2 JST PH2.0, J3 USB C 16P, Q1 DMG3415U, SW1 BOOT, SW2 RESET, SW3 MSK-12C02-07, U1 ESP32-C3-MINI-1, U2 Delta Board 2, U3 MCP73831T-2ACI/OT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

Commit message: Update for poduction
Parts:
- removed SW3: MSK-12C02-07, DeltaT32:MSK-12C02-07
- removed kibuzzard-680CDAE0: G***, kibuzzard-680CDAE0
- added D10: DNP, LED_SMD:LED_0603_1608Metric, F.Cu at (122.9, 104.9)
- added R21: 470R, Resistor_SMD:R_0402_1005Metric, F.Cu at (121.7, 103.5)
- added R22: 100, Resistor_SMD:R_0402_1005Metric, F.Cu at (114.4, 92.8)
- added kibuzzard-68198D94: G***, kibuzzard-68198D94, F.Cu at (123.5, 106.2)
- D3: value BLUE LED -> WHITE LED
- R16: value 22K1 -> 22K
Connections:
- C11 pad 1: /Switch -> +3V3
- C12 pad 1: /Switch -> +3V3
- L1 pad 2: /Switch -> +3V3
- R15 pad 2: /Switch -> +3V3
- R16 pad 2: Net-(U4-FB) -> Net-(R16-Pad2)
Routing:
- net /Switch: track 23.3 -> 0.00 mm, vias 2 -> 0
- net +3V3: track 89.5 -> 112.2 mm, vias 5 -> 7
- net Net-(D10-A): track 0.00 -> 1.40 mm
- net Net-(R16-Pad2): track 0.00 -> 1.13 mm
- net GND: vias 121 -> 120
- added copper zone on F.Cu, net +3V3
- removed copper zone on F.Cu, net /Switch
