File: hardware/esp-unit-c3-v3/esp-unit-c3-v3.kicad_sch (KiCad schematic)
At the start: 55 parts, among them J1 Conn_01x04, J2 JST PH2.0, J3 USB C 16P, Q1 DMG3415U, SW1 BOOT, SW2 RESET, SW3 MSK-12C02-07, U1 ESP32-C3-MINI-1, U2 Delta Board 2, U3 MCP73831T-2ACI/OT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

Commit message: Update for poduction
Parts:
- removed SW3: MSK-12C02-07, DeltaT32:MSK-12C02-07, symbol Switch:SW_SPDT_312
- added D10: DNP, LED_SMD:LED_0603_1608Metric, symbol Device:LED
- added R21: 470R, Resistor_SMD:R_0402_1005Metric, symbol Device:R
- added R22: 100, Resistor_SMD:R_0402_1005Metric, symbol Device:R
- D1: LCSC (none) -> C965555
- D3: LCSC C2286 -> C2288
- J3: LCSC (none) -> C165948; MANUFACTURER (none) -> GCT; MAXIMUM_PACKAGE_HEIGHT (none) -> 3.31 mm; PARTREV (none) -> A3; STANDARD (none) -> Manufacturer Recommendations
- R16: value 22K1 -> 22K; LCSC C43473 -> C25768
- R17: LCSC (none) -> C17699
- R18: LCSC (none) -> C17485
- U1: LCSC (none) -> C2838502
Connections:
- net Switch is gone; now on net +3V3: C11.1, C12.1, L1.2, R15.2
- net +3V3: now also R21.1
- net GND: now also D10.1 (K)
- net at C11.2, R15.1, U4.5 (FB): now also R22.1; no longer R16.2
- new net: D10.2 (A), R21.2
- new net: R16.2, R22.2
- no-connect marks 4 -> 3
Other:
- note added: "Buttons (Reset & Boot) Do Not Populate"
- note removed: "Buttons (Reset & Boot)"
