File: hardware/sensor-bmi-v2/sensor-bmi-v2.kicad_sch (KiCad schematic)
At the start: 24 parts, among them J1 JST SH1.0, Q1 BSS138, Q2 BSS138, U1 LN1134A182MR-G, U2 MAX30102, U3 LIS2MDL, U4 BMI160

Commit message: Update for poduction
Parts:
- removed C3: 100nF 16V, Capacitor_SMD:C_0603_1608Metric, symbol Device:C_Small
- removed R3, R6: 10K, Resistor_SMD:R_0402_1005Metric, symbol Device:R
- removed TP2: LIS_INT, TestPoint:TestPoint_Pad_D1.0mm, symbol Connector:TestPoint
- removed U3: LIS2MDL, Package_LGA:LGA-12_2x2mm_P0.5mm, symbol Sensor_Magnetic:LIS2MDL
- added C43: 100nF 10V, Capacitor_SMD:C_0603_1608Metric, symbol Device:C_Small
- added R43, R51: 10K, Resistor_SMD:R_0402_1005Metric, symbol Device:R
- added R50: DNP, Resistor_SMD:R_0402_1005Metric, symbol Device:R
- added TP42: LIS_INT, TestPoint:TestPoint_Pad_D1.0mm, symbol Connector:TestPoint
- added U45: LIS3MDL, Package_LGA:LGA-12_2x2mm_P0.5mm, symbol Sensor_Magnetic:LIS3MDL
- C41: renamed from C1; LCSC (none) -> C15849
- C42: renamed from C2; LCSC (none) -> C23630
- C44: renamed from C4; value 100nF 16V -> 100nF 10V; LCSC (none) -> C14663
- C45: renamed from C5; value 100nF 16V -> 100nF 10V; LCSC (none) -> C14663
- Q41: renamed from Q1; LCSC (none) -> C52895
- Q42: renamed from Q2; LCSC (none) -> C52895
- R41: renamed from R1; LCSC (none) -> C25744
- R42: renamed from R2; LCSC (none) -> C25744
- R44: renamed from R4; LCSC (none) -> C25744
- R45: renamed from R5; LCSC (none) -> C25744
- R47: renamed from R7; value 0R -> DNP
- R48: renamed from R8; LCSC (none) -> C25744
- R49: renamed from R9; LCSC (none) -> C25744
- U41: renamed from U1; LCSC (none) -> C141424
- U44: renamed from U4; value BMI160 -> BMI270; LCSC (none) -> C2836813
- renumbered J1 to J41, TP1 to TP41, TP3 to TP43, U2 to U42
Connections:
- net +3V3: now also R43.1, R50.1, U45.5 (Vdd), U45.6 (Vdd_IO)
- net GND: now also C43.2, R51.2, U45.12 (GND), U45.2 (GND), U45.3 (GND)
- net SCL: now also U45.1 (SCL/SPC)
- net SDA: now also U45.11 (SDA/SDI/SDO)
- new net: C43.1, U45.4 (C1)
- new net: R50.2, R51.1, U45.9 (SDO/SA1)
- new net: R43.2, U45.10 (~{CS})
- new net: TP42.1, U45.7 (INT)
- no-connect marks 6 -> 7
Other:
- note added: "LIS3MDL"
- note removed: "LIS2MDL"
