File: hardware/sensor-mpu-v2/sensor-mpu-v2.kicad_sch (KiCad schematic)
At the start: 20 parts, among them J1 JST SH1.0, Q1 BSS138, Q2 BSS138, U1 LN1134A182MR-G, U2 MPU-9250, U3 MAX30102

Commit message: Update for poduction
Parts:
- C81: renamed from C1; LCSC (none) -> C52923
- C82: renamed from C2; value 10nF 16V -> 10nF 10V; LCSC (none) -> C15195
- C83: renamed from C3; LCSC (none) -> C23630
- C84: renamed from C4; value 100nF 16V -> 100nF 10V; LCSC (none) -> C1525
- C85: renamed from C5; value 100nF 16V -> 100nF 10V; LCSC (none) -> C1525
- Q81: renamed from Q1; LCSC (none) -> C52895
- Q82: renamed from Q2; LCSC (none) -> C52895
- R81: renamed from R1; value 0R -> DNP
- R82: renamed from R2; LCSC (none) -> C25744
- R83: renamed from R3; LCSC (none) -> C25744
- R84: renamed from R4; LCSC (none) -> C25744
- R85: renamed from R5; LCSC (none) -> C25744
- R86: renamed from R6; LCSC (none) -> C25744
- U81: renamed from U1; LCSC (none) -> C141424
- renumbered J1 to J81, TP1 to TP81, TP2 to TP82, TP3 to TP83, U2 to U82, U3 to U83
